File: Z80_TestBoard.kicad_pcb (KiCad board)
At the start: 2 copper layers, 68.5 x 58 mm, 32 parts, among them J3 PWR, J5 CLK_SW, J7 USB_B_Mini, SW1 RESET, U1 Z84C00_PLCC, U2 NE555P

Commit message: add SOP28-DIP28 + LED-Board.
Parts:
- added C11: 100uF, Capacitor_THT:C_Radial_D4.0mm_H5.0mm_P1.50mm, F.Cu at (177.2, 133.9)
- added J1: LEFT, Connector_PinHeader_2.54mm:PinHeader_1x14_P2.54mm_Vertical, F.Cu at (148.5, 116.1)
- added J2: RIGHT, Connector_PinHeader_2.54mm:PinHeader_1x14_P2.54mm_Vertical, F.Cu at (148.5, 134.1)
- added J6: LED_01x03, Connector_PinHeader_2.54mm:PinHeader_1x03_P2.54mm_Vertical, F.Cu at (163.1, 116.5)
- added J8: USB_B_Mini, Connector_USB:USB_MINI_B_90_Angled, F.Cu at (175.0, 138.1)
- added SW2: ON|OFF, Button_Switch_THT:SW_Push_2P2T_Toggle_CK_PVA2OAH5xxxxxxV2, F.Cu at (168.5, 130.9)
- added SW3: PICK COLOR, Button_Switch_THT:SW_Slide-03_Wuerth-WS-SLTV_10x2.5x6.4_P2.54mm, F.Cu at (161.0, 143.4)
- added U3: IS65C256AL, Package_SO:SOP-28_8.4x18.16mm_P1.27mm, F.Cu at (132.1, 125.0)
- RV1: value 100K-POT -> POT
Connections:
- net /555_CLK renamed /Root/555_CLK
- net /A0 renamed /Root/A0
- net /A1 renamed /Root/A1
- net /A2 renamed /Root/A2
- net /A3 renamed /Root/A3
- net /A4 renamed /Root/A4
- net /A5 renamed /Root/A5
- net /A6 renamed /Root/A6
- net /A7 renamed /Root/A7
- net /BUSREQ renamed /Root/BUSREQ
- net /D0 renamed /Root/D0
- net /D1 renamed /Root/D1
- net /D2 renamed /Root/D2
- net /D3 renamed /Root/D3
- net /D4 renamed /Root/D4
- net /D5 renamed /Root/D5
- net /D6 renamed /Root/D6
- net /D7 renamed /Root/D7
- net /HALT renamed /Root/HALT
- net /INT renamed /Root/INT
- net /M1 renamed /Root/M1
- net /NMI renamed /Root/NMI
- net /RESET renamed /Root/RESET
- net /WAIT renamed /Root/WAIT
- net /Z80_CLK renamed /Root/Z80_CLK
Routing:
- net /LED_Board/LED_V1-: track 0.00 -> 30.3 mm, vias 0 -> 2
- net /LED_Board/LED_V2-: track 0.00 -> 28.9 mm
- net Net-(J8-VBUS): track 0.00 -> 25.0 mm
- net /SOP28-DIP28/IO_3: track 0.00 -> 9.77 mm
- net /SOP28-DIP28/GND3: track 0.00 -> 9.72 mm
- net /SOP28-DIP28/VCC3: track 0.00 -> 9.63 mm
- net /SOP28-DIP28/A14: track 0.00 -> 9.58 mm
- net /SOP28-DIP28/IO_4: track 0.00 -> 9.17 mm
- net /SOP28-DIP28/WE: track 0.00 -> 9.03 mm
- net /SOP28-DIP28/A12: track 0.00 -> 8.86 mm
- net /SOP28-DIP28/IO_2: track 0.00 -> 8.75 mm
- net /SOP28-DIP28/IO_5: track 0.00 -> 7.90 mm
- net /SOP28-DIP28/A13: track 0.00 -> 7.76 mm
- net /SOP28-DIP28/IO_1: track 0.00 -> 7.48 mm
- net /SOP28-DIP28/A7: track 0.00 -> 7.44 mm
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- added copper zone on B.Cu, net GND1
- added copper zone on F.Cu, net VCCQ
Other:
- board size 68.5 x 58 mm -> 68.5 x 91.9 mm
- board text added: "1"
- board text added: "15"
- board text added: "BOTTOM"
- board text added: "Board = 32x26 SW.Off = 14x7"
- board text added: "SOP28-DIP28"
- board text added: "TOP"
